Commit message: Added rviz files. Began fixing Dreamer demo.

File: dreamer_controlit/models/dreamer_controlit/xacro/dreamer_controlit_gazebo.xacro (robot description, xacro)
@@ -1,9 +1,184 @@
 <?xml version="1.0"?>
 <robot xmlns:xacro="http://ros.org/wiki/xacro" name="dreamer">
-    <xacro:include filename="$(find dreamer)/models/dreamer/xacro/dreamer_gazebo.xacro" />
+    <!-- Define the joint types. This specifies the joints that are simulated. -->
+    <property name="EYE_JOINT_TYPE" value="revolute" />
+    <property name="RIGHT_HAND_JOINT_TYPE" value="revolute" />
+    <property name="LEFT_GRIPPER_JOINT_TYPE" value="revolute" />
+    <property name="JOINT_TYPE_TORSO_YAW"               value="fixed" />
+    <property name="JOINT_TYPE_TORSO_LOWER_PITCH"       value="revolute" />
+    <property name="JOINT_TYPE_TORSO_UPPER_PITCH"       value="revolute" />
+    <property name="JOINT_TYPE_LOWER_NECK_PITCH"        value="revolute" />
+    <property name="JOINT_TYPE_UPPER_NECK_YAW"          value="revolute" />
+    <property name="JOINT_TYPE_UPPER_NECK_ROLL"         value="revolute" />
+    <property name="JOINT_TYPE_UPPER_NECK_PITCH"        value="revolute" />
+    <property name="JOINT_TYPE_LEFT_SHOULDER_EXTENSOR"  value="revolute" />
+    <property name="JOINT_TYPE_LEFT_SHOULDER_ABDUCTOR"  value="revolute" />
+    <property name="JOINT_TYPE_LEFT_SHOULDER_ROTATOR"   value="revolute" />
+    <property name="JOINT_TYPE_LEFT_ELBOW"              value="revolute" />
+    <property name="JOINT_TYPE_LEFT_WRIST_ROTATOR"      value="revolute" />
+    <property name="JOINT_TYPE_LEFT_WRIST_PITCH"        value="revolute" />
+    <property name="JOINT_TYPE_LEFT_WRIST_YAW"          value="revolute" />
+    <property name="JOINT_TYPE_RIGHT_SHOULDER_EXTENSOR" value="revolute" />
+    <property name="JOINT_TYPE_RIGHT_SHOULDER_ABDUCTOR" value="revolute" />
+    <property name="JOINT_TYPE_RIGHT_SHOULDER_ROTATOR"  value="revolute" />
+    <property name="JOINT_TYPE_RIGHT_ELBOW"             value="revolute" />
+    <property name="JOINT_TYPE_RIGHT_WRIST_ROTATOR"     value="revolute" />
+    <property name="JOINT_TYPE_RIGHT_WRIST_PITCH"       value="revolute" />
+    <property name="JOINT_TYPE_RIGHT_WRIST_YAW"         value="revolute" />
+    <property name="MESH_QUALITY" value="optimized" />
+    <property name="MESH_EXTENSION" value="stl" />
+    <!-- Gazebo uses "model:// for the model path -->
+    <property name="modelPath" value="model://dreamer" />
+    <property name="gripperModelPath" value="model://dreamer" />
+    <!-- Load the Dreamer Model -->
+    <xacro:include filename="$(find dreamer)/models/dreamer/xacro/dreamer_base.xacro" />
     <gazebo version="1.2">
+    	<!-- Pin the robot to the world -->
+    	<plugin filename="libPinPlugin.so" name="PinPlugin">
+            <pin_root_link>1</pin_root_link>
+        </plugin>
+        <!-- Enable shared memory communication between Gazebo and ControlIt! -->
         <plugin filename="libSMControlPlugin.so" name="SMControlPlugin">
             <node>/sm_control_plugin</node>
         </plugin>
+        <!-- Mimic the internal transmission in Dreamer's torso. -->
+        <plugin filename="libDreamerTorsoTransmissionPlugin.so" name="DreamerTorsoTransmissionPlugin"/>
+        <!-- Control the eyes. -->
+        <!-- <plugin filename="libdreamer_eye_plugin.so" name="DreamerEyePlugin"/> -->
+        <!-- Control the right hand. -->
+        <!-- <plugin filename="libdreamer_hand_poscom_plugin.so" name="RightHandPosComPlugin"/> -->
+        <!-- Control the left gripper. -->
+        <!-- <plugin filename="libdreamer_pr2_gripper_plugin.so" name="DreamerGripperPlugin"/> -->
+    </gazebo>
+    <!--
+      The following enables torque feedback.  Without these, the following warning will be printed
+      by Gazebo when the shared memory plugin is used:
+      Warning [ODEJoint.cc:1105] GetForceTorque: forgot to set <provide_feedback>?
+    -->
+    <!-- Torso joints -->
+    <gazebo reference="torso_yaw">
+        <provideFeedback value="true"/>
+    </gazebo>
+    <gazebo reference="torso_lower_pitch">
+        <provideFeedback value="true"/>
+    </gazebo>
+    <gazebo reference="torso_upper_pitch">
+        <provideFeedback value="true"/>
+    </gazebo>
+    <!-- right arm joints -->
+    <gazebo reference="right_shoulder_extensor">
+        <provideFeedback value="true"/>
+    </gazebo>
+    <gazebo reference="right_shoulder_abductor">
+        <provideFeedback value="true"/>
+    </gazebo>
+    <gazebo reference="right_shoulder_rotator">
+        <provideFeedback value="true"/>
+    </gazebo>
+    <gazebo reference="right_elbow">
+        <provideFeedback value="true"/>
+    </gazebo>
+    <gazebo reference="right_wrist_rotator">
+        <provideFeedback value="true"/>
+    </gazebo>
+    <gazebo reference="right_wrist_pitch">
+        <provideFeedback value="true"/>
+    </gazebo>
+    <gazebo reference="right_wrist_yaw">
+        <provideFeedback value="true"/>
+    </gazebo>
+    <!-- Left arm joints -->
+    <gazebo reference="left_shoulder_extensor">
+        <provideFeedback value="true"/>
+    </gazebo>
+    <gazebo reference="left_shoulder_abductor">
+        <provideFeedback value="true"/>
+    </gazebo>
+    <gazebo reference="left_shoulder_rotator">
+        <provideFeedback value="true"/>
+    </gazebo>
+    <gazebo reference="left_elbow">
+        <provideFeedback value="true"/>
+    </gazebo>
+    <gazebo reference="left_wrist_rotator">
+        <provideFeedback value="true"/>
+    </gazebo>
+    <gazebo reference="left_wrist_pitch">
+        <provideFeedback value="true"/>
+    </gazebo>
+    <gazebo reference="left_wrist_yaw">
+        <provideFeedback value="true"/>
+    </gazebo>
+    <!-- Head and neck joints -->
+    <gazebo reference="lower_neck_pitch">
+        <provideFeedback value="true"/>
+    </gazebo>
+    <gazebo reference="upper_neck_yaw">
+        <provideFeedback value="true"/>
+    </gazebo>
+    <gazebo reference="upper_neck_roll">
+        <provideFeedback value="true"/>
+    </gazebo>
+    <gazebo reference="upper_neck_pitch">
+        <provideFeedback value="true"/>
+    </gazebo>
+    <gazebo reference="eye_pitch">
+        <provideFeedback value="true"/>
+    </gazebo>
+    <gazebo reference="right_eye_yaw">
+        <provideFeedback value="true"/>
+    </gazebo>
+    <gazebo reference="left_eye_yaw">
+        <provideFeedback value="true"/>
+    </gazebo>
+    <!-- Right hand joints -->
+    <gazebo reference="right_thumb_1">
+        <provideFeedback value="true"/>
+    </gazebo>
+    <gazebo reference="right_thumb_2">
+        <provideFeedback value="true"/>
+    </gazebo>
+    <gazebo reference="right_thumb_3">
+        <provideFeedback value="true"/>
+    </gazebo>
+    <gazebo reference="right_pointer_finger_1">
+        <provideFeedback value="true"/>
+    </gazebo>
+    <gazebo reference="right_pointer_finger_2">
+        <provideFeedback value="true"/>
+    </gazebo>
+    <gazebo reference="right_pointer_finger_3">
+        <provideFeedback value="true"/>
+    </gazebo>
+    <gazebo reference="right_middle_finger_1">
+        <provideFeedback value="true"/>
+    </gazebo>
+    <gazebo reference="right_middle_finger_2">
+        <provideFeedback value="true"/>
+    </gazebo>
+    <gazebo reference="right_middle_finger_3">
+        <provideFeedback value="true"/>
+    </gazebo>
+    <gazebo reference="right_pinky_1">
+        <provideFeedback value="true"/>
+    </gazebo>
+    <gazebo reference="right_pinky_2">
+        <provideFeedback value="true"/>
+    </gazebo>
+    <gazebo reference="right_pinky_3">
+        <provideFeedback value="true"/>
+    </gazebo>
+    <!-- Left gripper joints -->
+    <gazebo reference="l_gripper_l_finger_joint">
+        <provideFeedback value="true"/>
+    </gazebo>
+    <gazebo reference="l_gripper_l_finger_tip_joint">
+        <provideFeedback value="true"/>
+    </gazebo>
+    <gazebo reference="l_gripper_r_finger_joint">
+        <provideFeedback value="true"/>
+    </gazebo>
+    <gazebo reference="l_gripper_r_finger_tip_joint">
+        <provideFeedback value="true"/>
     </gazebo>
 </robot>

File: dreamer_controlit/models/dreamer_controlit/xacro/dreamer_controlit_rviz.xacro (robot description, xacro)
@@ -26,4 +26,6 @@
     <property name="JOINT_TYPE_RIGHT_WRIST_PITCH"       value="revolute" />
     <property name="JOINT_TYPE_RIGHT_WRIST_YAW"         value="revolute" />
+    <property name="MESH_QUALITY" value="optimized" />
+    <property name="MESH_EXTENSION" value="stl" />
     <!-- RViz uses package:// for the model path -->
     <property name="modelPath" value="package://dreamer/models/dreamer" />

File: dreamer_testbed_controlit/models/dreamer_testbed_controlit/urdf/dreamer_testbed_gazebo.urdf (robot description, URDF)
Before this commit: robot dreamer, 46 links, 45 joints
Links:
- added link camera_arm0, mass 0.267875; collision box size=0.25 0.04 0.04; visual box size=0.25 0.04 0.04
- added link camera_arm1, mass 1.125075; collision box size=0.04 0.04 1.05; visual box size=0.04 0.04 1.05
- added link camera_arm2, mass 0.696475; collision box size=0.65 0.04 0.04; visual box size=0.65 0.04 0.04
- added link camera_arm3, mass 0.10715; collision box size=0.04 0.04 0.1; visual box size=0.04 0.04 0.1
- added link camera_link1, mass 0.01; collision box size=0.08 0.02 0.02; visual box size=0.08 0.02 0.02
- added link camera_link2, mass 0.01; collision box size=0.08 0.02 0.02; visual box size=0.08 0.02 0.02
- added link testbed_base, mass 20; collision box size=0.8 0.5 0.05; visual box size=0.8 0.5 0.05
- added link testbed_stand, mass 20; collision box size=0.25 0.25 0.8; visual box size=0.25 0.25 0.8
- added link webcam1_virtual_link, mass 0.01
- added link webcam2_virtual_link, mass 0.01
- link l_gripper_l_finger_link: geometry collision mesh filename=package://dreamer/models/dreamer/meka_description/meshes/gr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; visual mesh filename=package://dreamer/models/dreamer/meka_description/meshes/gr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
- link l_gripper_l_finger_tip_link: geometry collision mesh filename=package://dreamer/models/dreamer/meka_description/meshes/gr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; visual mesh filename=package://dreamer/models/dreamer/meka_description/meshes/gr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
- link l_gripper_palm_link: geometry collision mesh filename=package://dreamer/models/dreamer/meka_description/meshes/gr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; visual mesh filename=package://dreamer/models/dreamer/meka_description/meshes/gr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
- link l_gripper_r_finger_link: geometry collision mesh filename=package://dreamer/models/dreamer/meka_description/meshes/gr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; visual mesh filename=package://dreamer/models/dreamer/meka_description/meshes/gr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
- link l_gripper_r_finger_tip_link: geometry collision mesh filename=package://dreamer/models/dreamer/meka_description/meshes/gr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; visual mesh filename=package://dreamer/models/dreamer/meka_description/meshes/gr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
Joints:
- added joint base_to_stand: type fixed, parent testbed_base, child testbed_stand, origin xyz=0.0 0 0.01 rpy=0 0 0
- added joint fixed0: type fixed, parent testbed_stand, child camera_arm0, origin xyz=-0.12 0 0.8 rpy=0 0 0
- added joint fixed1: type fixed, parent camera_arm0, child camera_arm1, origin xyz=-0.23095 0 0 rpy=0 0 0
- added joint fixed2: type fixed, parent camera_arm1, child camera_arm2, origin xyz=0 0 1.03095 rpy=0 0 0
- added joint fixed3: type fixed, parent camera_arm2, child camera_arm3, origin xyz=0.63095 0 0 rpy=0 0 0
- added joint testbed_base_offset: type fixed, parent panplate_link, child testbed_base, origin xyz=0.0 0.0 0.0 rpy=0 0 0
- added joint webcam1_mount_x: type continuous, parent webcam1_virtual_link, child camera_link1, origin xyz=0 0.005 0.0 rpy=0.0 0 0, axis 0 0 1
- added joint webcam1_mount_y: type continuous, parent camera_arm3, child webcam1_virtual_link, origin xyz=0 0.05 -0.1 rpy=0.0 0 0, axis 0 1 0
- added joint webcam2_mount_x: type continuous, parent webcam2_virtual_link, child camera_link2, origin xyz=0 -0.005 0.0 rpy=0.0 0.0 0.0, axis 0 0 1
- added joint webcam2_mount_y: type continuous, parent camera_arm3, child webcam2_virtual_link, origin xyz=0 -0.05 -0.1 rpy=0.0 0.0 0.0, axis 0 1 0
- joint eye_pitch: type revolute -> fixed
- joint left_eye_yaw: type revolute -> fixed
- joint lower_neck_pitch: type revolute -> fixed
- joint right_eye_yaw: type revolute -> fixed
- joint upper_neck_pitch: type revolute -> fixed
- joint upper_neck_roll: type revolute -> fixed
- joint upper_neck_yaw: type revolute -> fixed

File: dreamer_testbed_controlit/models/dreamer_testbed_controlit/xacro/dreamer_testbed_gazebo.xacro (robot description, xacro)
@@ -26,4 +26,6 @@
     <property name="JOINT_TYPE_RIGHT_WRIST_PITCH"       value="revolute" />
     <property name="JOINT_TYPE_RIGHT_WRIST_YAW"         value="revolute" />
+    <property name="MESH_QUALITY" value="optimized" />
+    <property name="MESH_EXTENSION" value="stl" />
     <!-- Gazebo uses model:// for the model path. -->
     <property name="modelPath" value="model://dreamer" />
