Commit message: xacro style guide

File: atlas_legs_plain_controlit/models/atlas_legs_plain_controlit/xacro/atlas_legs_plain_controlit.xacro (robot description, xacro)
@@ -1,5 +1,5 @@
 <robot xmlns:xacro="http://www.ros.org/wiki/xacro" name="atlas_legs_plain" >
 	<!-- rViz uses package:// for the model path. -->
-    <property name="modelPath" value="package://atlas_plain/models/atlas_plain" />
+    <xacro:property name="modelPath" value="package://atlas_plain/models/atlas_plain" />
     <xacro:include filename="$(find atlas_legs_plain)/models/atlas_legs_plain/xacro/atlas_legs_plain_base.xacro" />
     <atlas_legs_plain />

File: atlas_plain_controlit/models/atlas_plain_controlit/xacro/atlas_plain_with_sandia_hands_controlit.xacro (robot description, xacro)
@@ -1,5 +1,5 @@
 <robot xmlns:xacro="http://www.ros.org/wiki/xacro" name="atlas" >
     <!-- rViz uses package:// for the model path. -->
-    <property name="modelPath" value="package://atlas_plain/models/atlas_plain" />
+    <xacro:property name="modelPath" value="package://atlas_plain/models/atlas_plain" />
     <xacro:include filename="$(find atlas_plain)/models/atlas_plain/xacro/atlas_plain_base.xacro" />
     <xacro:include filename="$(find atlas_plain)/models/sandia_hands/xacro/sandia_hand_simple_shapes.urdf.xacro" />

File: atlas_plain_controlit/models/atlas_plain_controlit/xacro/atlas_plain_with_sandia_hands_gazebo.xacro (robot description, xacro)
@@ -1,5 +1,5 @@
 <robot xmlns:xacro="http://www.ros.org/wiki/xacro" name="atlas" >
     <!-- gazebo uses model:// for the model path. -->
-    <property name="modelPath" value="model://atlas_plain" />
+    <xacro:property name="modelPath" value="model://atlas_plain" />
     <xacro:include filename="$(find atlas_plain)/models/atlas_plain/xacro/atlas_plain_with_sandia_hands.xacro" />
     <gazebo>

File: atlas_plain_pinned_controlit/models/atlas_plain_pinned_controlit/xacro/atlas_plain_pinned_controlit.xacro (robot description, xacro)
@@ -1,5 +1,5 @@
 <robot xmlns:xacro="http://www.ros.org/wiki/xacro" name="atlas" >
     <!-- rViz uses package:// for the model path. -->
-    <property name="modelPath" value="package://atlas_plain/models/atlas_plain" />
+    <xacro:property name="modelPath" value="package://atlas_plain/models/atlas_plain" />
     <xacro:include filename="$(find atlas_plain)/models/atlas_plain/xacro/atlas_plain_base.xacro" />
     <!-- <xacro:include filename="$(find atlas_plain)/models/sandia_hands/xacro/sandia_hand_simple_shapes.urdf.xacro" /> -->

File: atlas_plain_pinned_controlit/models/atlas_plain_pinned_controlit/xacro/atlas_plain_pinned_gazebo.xacro (robot description, xacro)
@@ -1,5 +1,5 @@
 <robot xmlns:xacro="http://www.ros.org/wiki/xacro" name="atlas_legs_plain" >
     <!-- gazebo uses model:// for the model path. -->
-    <property name="modelPath" value="model://atlas_plain" />
+    <xacro:property name="modelPath" value="model://atlas_plain" />
     <xacro:include filename="$(find atlas_plain_pinned)/models/atlas_plain_pinned/xacro/atlas_plain_pinned.xacro" />
     <gazebo version="1.2">

File: dreamer_controlit/models/dreamer_controlit/xacro/dreamer_controlit_gazebo.xacro (robot description, xacro)
@@ -2,33 +2,33 @@
 <robot xmlns:xacro="http://ros.org/wiki/xacro" name="dreamer">
     <!-- Define the joint types. This specifies the joints that are simulated. -->
-    <property name="EYE_JOINT_TYPE" value="revolute" />
-    <property name="RIGHT_HAND_JOINT_TYPE" value="revolute" />
-    <property name="LEFT_GRIPPER_JOINT_TYPE" value="revolute" />
-    <property name="JOINT_TYPE_TORSO_YAW"               value="fixed" />
-    <property name="JOINT_TYPE_TORSO_LOWER_PITCH"       value="revolute" />
-    <property name="JOINT_TYPE_TORSO_UPPER_PITCH"       value="revolute" />
-    <property name="JOINT_TYPE_LOWER_NECK_PITCH"        value="revolute" />
-    <property name="JOINT_TYPE_UPPER_NECK_YAW"          value="revolute" />
-    <property name="JOINT_TYPE_UPPER_NECK_ROLL"         value="revolute" />
-    <property name="JOINT_TYPE_UPPER_NECK_PITCH"        value="revolute" />
-    <property name="JOINT_TYPE_LEFT_SHOULDER_EXTENSOR"  value="revolute" />
-    <property name="JOINT_TYPE_LEFT_SHOULDER_ABDUCTOR"  value="revolute" />
-    <property name="JOINT_TYPE_LEFT_SHOULDER_ROTATOR"   value="revolute" />
-    <property name="JOINT_TYPE_LEFT_ELBOW"              value="revolute" />
-    <property name="JOINT_TYPE_LEFT_WRIST_ROTATOR"      value="revolute" />
-    <property name="JOINT_TYPE_LEFT_WRIST_PITCH"        value="revolute" />
-    <property name="JOINT_TYPE_LEFT_WRIST_YAW"          value="revolute" />
-    <property name="JOINT_TYPE_RIGHT_SHOULDER_EXTENSOR" value="revolute" />
-    <property name="JOINT_TYPE_RIGHT_SHOULDER_ABDUCTOR" value="revolute" />
-    <property name="JOINT_TYPE_RIGHT_SHOULDER_ROTATOR"  value="revolute" />
-    <property name="JOINT_TYPE_RIGHT_ELBOW"             value="revolute" />
-    <property name="JOINT_TYPE_RIGHT_WRIST_ROTATOR"     value="revolute" />
-    <property name="JOINT_TYPE_RIGHT_WRIST_PITCH"       value="revolute" />
-    <property name="JOINT_TYPE_RIGHT_WRIST_YAW"         value="revolute" />
-    <property name="MESH_QUALITY" value="optimized" />
-    <property name="MESH_EXTENSION" value="stl" />
+    <xacro:property name="EYE_JOINT_TYPE" value="revolute" />
+    <xacro:property name="RIGHT_HAND_JOINT_TYPE" value="revolute" />
+    <xacro:property name="LEFT_GRIPPER_JOINT_TYPE" value="revolute" />
+    <xacro:property name="JOINT_TYPE_TORSO_YAW"               value="fixed" />
+    <xacro:property name="JOINT_TYPE_TORSO_LOWER_PITCH"       value="revolute" />
+    <xacro:property name="JOINT_TYPE_TORSO_UPPER_PITCH"       value="revolute" />
+    <xacro:property name="JOINT_TYPE_LOWER_NECK_PITCH"        value="revolute" />
+    <xacro:property name="JOINT_TYPE_UPPER_NECK_YAW"          value="revolute" />
+    <xacro:property name="JOINT_TYPE_UPPER_NECK_ROLL"         value="revolute" />
+    <xacro:property name="JOINT_TYPE_UPPER_NECK_PITCH"        value="revolute" />
+    <xacro:property name="JOINT_TYPE_LEFT_SHOULDER_EXTENSOR"  value="revolute" />
+    <xacro:property name="JOINT_TYPE_LEFT_SHOULDER_ABDUCTOR"  value="revolute" />
+    <xacro:property name="JOINT_TYPE_LEFT_SHOULDER_ROTATOR"   value="revolute" />
+    <xacro:property name="JOINT_TYPE_LEFT_ELBOW"              value="revolute" />
+    <xacro:property name="JOINT_TYPE_LEFT_WRIST_ROTATOR"      value="revolute" />
+    <xacro:property name="JOINT_TYPE_LEFT_WRIST_PITCH"        value="revolute" />
+    <xacro:property name="JOINT_TYPE_LEFT_WRIST_YAW"          value="revolute" />
+    <xacro:property name="JOINT_TYPE_RIGHT_SHOULDER_EXTENSOR" value="revolute" />
+    <xacro:property name="JOINT_TYPE_RIGHT_SHOULDER_ABDUCTOR" value="revolute" />
+    <xacro:property name="JOINT_TYPE_RIGHT_SHOULDER_ROTATOR"  value="revolute" />
+    <xacro:property name="JOINT_TYPE_RIGHT_ELBOW"             value="revolute" />
+    <xacro:property name="JOINT_TYPE_RIGHT_WRIST_ROTATOR"     value="revolute" />
+    <xacro:property name="JOINT_TYPE_RIGHT_WRIST_PITCH"       value="revolute" />
+    <xacro:property name="JOINT_TYPE_RIGHT_WRIST_YAW"         value="revolute" />
+    <xacro:property name="MESH_QUALITY" value="optimized" />
+    <xacro:property name="MESH_EXTENSION" value="stl" />
     <!-- Gazebo uses "model:// for the model path -->
-    <property name="modelPath" value="model://dreamer" />
-    <property name="gripperModelPath" value="model://dreamer" />
+    <xacro:property name="modelPath" value="model://dreamer" />
+    <xacro:property name="gripperModelPath" value="model://dreamer" />
     <!-- Load the Dreamer Model -->
     <xacro:include filename="$(find dreamer)/models/dreamer/xacro/dreamer_base.xacro" />

File: dreamer_controlit/models/dreamer_controlit/xacro/dreamer_controlit_rviz.xacro (robot description, xacro)
@@ -2,33 +2,33 @@
 <robot xmlns:xacro="http://ros.org/wiki/xacro" name="dreamer">
     <!-- Define the joint types. This specifies the joints that are controlled by WBOSC. -->
-    <property name="EYE_JOINT_TYPE" value="fixed" />
-    <property name="RIGHT_HAND_JOINT_TYPE" value="fixed" />
-    <property name="LEFT_GRIPPER_JOINT_TYPE" value="fixed" />
-    <property name="JOINT_TYPE_TORSO_YAW"               value="fixed" />
-    <property name="JOINT_TYPE_TORSO_LOWER_PITCH"       value="revolute" />
-    <property name="JOINT_TYPE_TORSO_UPPER_PITCH"       value="revolute" />
-    <property name="JOINT_TYPE_LOWER_NECK_PITCH"        value="fixed" />
-    <property name="JOINT_TYPE_UPPER_NECK_YAW"          value="fixed" />
-    <property name="JOINT_TYPE_UPPER_NECK_ROLL"         value="fixed" />
-    <property name="JOINT_TYPE_UPPER_NECK_PITCH"        value="fixed" />
-    <property name="JOINT_TYPE_LEFT_SHOULDER_EXTENSOR"  value="revolute" />
-    <property name="JOINT_TYPE_LEFT_SHOULDER_ABDUCTOR"  value="revolute" />
-    <property name="JOINT_TYPE_LEFT_SHOULDER_ROTATOR"   value="revolute" />
-    <property name="JOINT_TYPE_LEFT_ELBOW"              value="revolute" />
-    <property name="JOINT_TYPE_LEFT_WRIST_ROTATOR"      value="revolute" />
-    <property name="JOINT_TYPE_LEFT_WRIST_PITCH"        value="revolute" />
-    <property name="JOINT_TYPE_LEFT_WRIST_YAW"          value="revolute" />
-    <property name="JOINT_TYPE_RIGHT_SHOULDER_EXTENSOR" value="revolute" />
-    <property name="JOINT_TYPE_RIGHT_SHOULDER_ABDUCTOR" value="revolute" />
-    <property name="JOINT_TYPE_RIGHT_SHOULDER_ROTATOR"  value="revolute" />
-    <property name="JOINT_TYPE_RIGHT_ELBOW"             value="revolute" />
-    <property name="JOINT_TYPE_RIGHT_WRIST_ROTATOR"     value="revolute" />
-    <property name="JOINT_TYPE_RIGHT_WRIST_PITCH"       value="revolute" />
-    <property name="JOINT_TYPE_RIGHT_WRIST_YAW"         value="revolute" />
-    <property name="MESH_QUALITY" value="optimized" />
-    <property name="MESH_EXTENSION" value="stl" />
+    <xacro:property name="EYE_JOINT_TYPE" value="fixed" />
+    <xacro:property name="RIGHT_HAND_JOINT_TYPE" value="fixed" />
+    <xacro:property name="LEFT_GRIPPER_JOINT_TYPE" value="fixed" />
+    <xacro:property name="JOINT_TYPE_TORSO_YAW"               value="fixed" />
+    <xacro:property name="JOINT_TYPE_TORSO_LOWER_PITCH"       value="revolute" />
+    <xacro:property name="JOINT_TYPE_TORSO_UPPER_PITCH"       value="revolute" />
+    <xacro:property name="JOINT_TYPE_LOWER_NECK_PITCH"        value="fixed" />
+    <xacro:property name="JOINT_TYPE_UPPER_NECK_YAW"          value="fixed" />
+    <xacro:property name="JOINT_TYPE_UPPER_NECK_ROLL"         value="fixed" />
+    <xacro:property name="JOINT_TYPE_UPPER_NECK_PITCH"        value="fixed" />
+    <xacro:property name="JOINT_TYPE_LEFT_SHOULDER_EXTENSOR"  value="revolute" />
+    <xacro:property name="JOINT_TYPE_LEFT_SHOULDER_ABDUCTOR"  value="revolute" />
+    <xacro:property name="JOINT_TYPE_LEFT_SHOULDER_ROTATOR"   value="revolute" />
+    <xacro:property name="JOINT_TYPE_LEFT_ELBOW"              value="revolute" />
+    <xacro:property name="JOINT_TYPE_LEFT_WRIST_ROTATOR"      value="revolute" />
+    <xacro:property name="JOINT_TYPE_LEFT_WRIST_PITCH"        value="revolute" />
+    <xacro:property name="JOINT_TYPE_LEFT_WRIST_YAW"          value="revolute" />
+    <xacro:property name="JOINT_TYPE_RIGHT_SHOULDER_EXTENSOR" value="revolute" />
+    <xacro:property name="JOINT_TYPE_RIGHT_SHOULDER_ABDUCTOR" value="revolute" />
+    <xacro:property name="JOINT_TYPE_RIGHT_SHOULDER_ROTATOR"  value="revolute" />
+    <xacro:property name="JOINT_TYPE_RIGHT_ELBOW"             value="revolute" />
+    <xacro:property name="JOINT_TYPE_RIGHT_WRIST_ROTATOR"     value="revolute" />
+    <xacro:property name="JOINT_TYPE_RIGHT_WRIST_PITCH"       value="revolute" />
+    <xacro:property name="JOINT_TYPE_RIGHT_WRIST_YAW"         value="revolute" />
+    <xacro:property name="MESH_QUALITY" value="optimized" />
+    <xacro:property name="MESH_EXTENSION" value="stl" />
     <!-- RViz uses package:// for the model path -->
-    <property name="modelPath" value="package://dreamer/models/dreamer" />
-    <property name="gripperModelPath" value="package://dreamer/models/dreamer" />
+    <xacro:property name="modelPath" value="package://dreamer/models/dreamer" />
+    <xacro:property name="gripperModelPath" value="package://dreamer/models/dreamer" />
     <!-- Load the Dreamer Model -->
     <xacro:include filename="$(find dreamer)/models/dreamer/xacro/dreamer_base.xacro" />

File: dreamer_testbed_controlit/models/dreamer_testbed_controlit/xacro/dreamer_testbed_gazebo.xacro (robot description, xacro)
@@ -2,32 +2,32 @@
 <robot xmlns:xacro="http://ros.org/wiki/xacro" name="dreamer_testbed">
     <!-- Define the joint types. This specifies the joints that are controlled by WBOSC. -->
-    <property name="EYE_JOINT_TYPE" value="fixed" />
-    <property name="RIGHT_HAND_JOINT_TYPE" value="revolute" />
-    <property name="LEFT_GRIPPER_JOINT_TYPE" value="revolute" />
-    <property name="JOINT_TYPE_TORSO_YAW"               value="fixed" />
-    <property name="JOINT_TYPE_TORSO_LOWER_PITCH"       value="revolute" />
-    <property name="JOINT_TYPE_TORSO_UPPER_PITCH"       value="revolute" />
-    <property name="JOINT_TYPE_LOWER_NECK_PITCH"        value="fixed" />
-    <property name="JOINT_TYPE_UPPER_NECK_YAW"          value="fixed" />
-    <property name="JOINT_TYPE_UPPER_NECK_ROLL"         value="fixed" />
-    <property name="JOINT_TYPE_UPPER_NECK_PITCH"        value="fixed" />
-    <property name="JOINT_TYPE_LEFT_SHOULDER_EXTENSOR"  value="revolute" />
-    <property name="JOINT_TYPE_LEFT_SHOULDER_ABDUCTOR"  value="revolute" />
-    <property name="JOINT_TYPE_LEFT_SHOULDER_ROTATOR"   value="revolute" />
-    <property name="JOINT_TYPE_LEFT_ELBOW"              value="revolute" />
-    <property name="JOINT_TYPE_LEFT_WRIST_ROTATOR"      value="revolute" />
-    <property name="JOINT_TYPE_LEFT_WRIST_PITCH"        value="revolute" />
-    <property name="JOINT_TYPE_LEFT_WRIST_YAW"          value="revolute" />
-    <property name="JOINT_TYPE_RIGHT_SHOULDER_EXTENSOR" value="revolute" />
-    <property name="JOINT_TYPE_RIGHT_SHOULDER_ABDUCTOR" value="revolute" />
-    <property name="JOINT_TYPE_RIGHT_SHOULDER_ROTATOR"  value="revolute" />
-    <property name="JOINT_TYPE_RIGHT_ELBOW"             value="revolute" />
-    <property name="JOINT_TYPE_RIGHT_WRIST_ROTATOR"     value="revolute" />
-    <property name="JOINT_TYPE_RIGHT_WRIST_PITCH"       value="revolute" />
-    <property name="JOINT_TYPE_RIGHT_WRIST_YAW"         value="revolute" />
-    <property name="MESH_QUALITY" value="optimized" />
-    <property name="MESH_EXTENSION" value="stl" />
+    <xacro:property name="EYE_JOINT_TYPE" value="fixed" />
+    <xacro:property name="RIGHT_HAND_JOINT_TYPE" value="revolute" />
+    <xacro:property name="LEFT_GRIPPER_JOINT_TYPE" value="revolute" />
+    <xacro:property name="JOINT_TYPE_TORSO_YAW"               value="fixed" />
+    <xacro:property name="JOINT_TYPE_TORSO_LOWER_PITCH"       value="revolute" />
+    <xacro:property name="JOINT_TYPE_TORSO_UPPER_PITCH"       value="revolute" />
+    <xacro:property name="JOINT_TYPE_LOWER_NECK_PITCH"        value="fixed" />
+    <xacro:property name="JOINT_TYPE_UPPER_NECK_YAW"          value="fixed" />
+    <xacro:property name="JOINT_TYPE_UPPER_NECK_ROLL"         value="fixed" />
+    <xacro:property name="JOINT_TYPE_UPPER_NECK_PITCH"        value="fixed" />
+    <xacro:property name="JOINT_TYPE_LEFT_SHOULDER_EXTENSOR"  value="revolute" />
+    <xacro:property name="JOINT_TYPE_LEFT_SHOULDER_ABDUCTOR"  value="revolute" />
+    <xacro:property name="JOINT_TYPE_LEFT_SHOULDER_ROTATOR"   value="revolute" />
+    <xacro:property name="JOINT_TYPE_LEFT_ELBOW"              value="revolute" />
+    <xacro:property name="JOINT_TYPE_LEFT_WRIST_ROTATOR"      value="revolute" />
+    <xacro:property name="JOINT_TYPE_LEFT_WRIST_PITCH"        value="revolute" />
+    <xacro:property name="JOINT_TYPE_LEFT_WRIST_YAW"          value="revolute" />
+    <xacro:property name="JOINT_TYPE_RIGHT_SHOULDER_EXTENSOR" value="revolute" />
+    <xacro:property name="JOINT_TYPE_RIGHT_SHOULDER_ABDUCTOR" value="revolute" />
+    <xacro:property name="JOINT_TYPE_RIGHT_SHOULDER_ROTATOR"  value="revolute" />
+    <xacro:property name="JOINT_TYPE_RIGHT_ELBOW"             value="revolute" />
+    <xacro:property name="JOINT_TYPE_RIGHT_WRIST_ROTATOR"     value="revolute" />
+    <xacro:property name="JOINT_TYPE_RIGHT_WRIST_PITCH"       value="revolute" />
+    <xacro:property name="JOINT_TYPE_RIGHT_WRIST_YAW"         value="revolute" />
+    <xacro:property name="MESH_QUALITY" value="optimized" />
+    <xacro:property name="MESH_EXTENSION" value="stl" />
     <!-- Gazebo uses model:// for the model path. -->
-    <property name="modelPath" value="model://dreamer" />
+    <xacro:property name="modelPath" value="model://dreamer" />
     <xacro:include filename="$(find dreamer_testbed)/models/dreamer_testbed/xacro/dreamer_testbed_base.xacro" />
     <gazebo version='1.2'>

File: valkyrie_upperbody_controlit/models/valkyrie_upperbody_controlit/xacro/valkyrie_upperbody_controlit.xacro (robot description, xacro)
@@ -2,5 +2,5 @@
 <robot xmlns:xacro="http://ros.org/wiki/xacro" name="dreamer">
     <!-- RViz uses package:// for the model path. -->
-    <property name="modelPath" value="package://valkyrie/models/valkyrie" />
+    <xacro:property name="modelPath" value="package://valkyrie/models/valkyrie" />
     <xacro:include filename="$(find valkyrie)/models/valkyrie/xacro/valkyrie_colors.xacro" />
     <xacro:include filename="$(find valkyrie)/models/valkyrie/xacro/valkyrie_upperbody_base.xacro" />
